File: kicad/ECP5.kicad_pcb (KiCad board)
At the start: 4 copper layers, 64.4 x 54.6 mm, 79 parts, among them J1 FLE-126-01-G-DV, J2 RCJ-044, J3 HDMI A, SW1 PTS645SK43SMTR92 LFS, T1 DA101JC, U3 74HC04, U4 DSLVDS1047

Commit message: Updated PCB
Parts:
- renumbered C4 to C1, C5 to C2, C6 to C3, C8 to C4, U3 to U1, U4 to U2
Changed lines of the file:
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@@
 	(net 55 "Net-(D8-K)")
 	(net 56 "+3V3")
-	(net 57 "Net-(C6-Pad2)")
+	(net 57 "Net-(C3-Pad2)")
 	(net 58 "Net-(R26-Pad2)")
 	(net 59 "Net-(J2-In)")
@@
 	(net 93 "DIFF_LRCK-")
 	(net 94 "unconnected-(J3-HPD-Pad19)")
-	(net 95 "Net-(U3-Pad2)")
-	(net 96 "unconnected-(U3-Pad10)")
-	(net 97 "unconnected-(U3-Pad12)")
-	(net 98 "unconnected-(U3-Pad8)")
+	(net 95 "Net-(U1-Pad2)")
+	(net 96 "unconnected-(U1-Pad10)")
+	(net 97 "unconnected-(U1-Pad12)")
+	(net 98 "unconnected-(U1-Pad8)")
 	(footprint "LED_SMD:LED_0603_1608Metric"
 		(layer "F.Cu")
@@
 			(size 3 1.5)
 			(layers "F.Cu" "F.Paste" "F.Mask")
-			(net 57 "Net-(C6-Pad2)")
+			(net 57 "Net-(C3-Pad2)")
 			(pinfunction "1")
 			(pintype "passive")
@@
 			(layers "F.Cu" "F.Paste" "F.Mask")
 			(roundrect_rratio 0.25)
-			(net 57 "Net-(C6-Pad2)")
+			(net 57 "Net-(C3-Pad2)")
 			(pintype "passive")
 		)
@@
 		(descr "Capacitor SMD 0603 (1608 Metric), square (rectangular) end terminal, IPC_7351 nominal, (Body size source: IPC-SM-782 page 76, https://www.pcb-3d.com/wordpress/wp-content/uploads/ipc-sm-782a_amendment_1_and_2.pdf), generated with kicad-footprint-generator")
 		(tags "capacitor")
-		(property "Reference" "C6"
+		(property "Reference" "C3"
 			(at 0 1.15 90)
 			(unlocked yes)
@@
 			(layers "F.Cu" "F.Paste" "F.Mask")
 			(roundrect_rratio 0.25)
-			(net 57 "Net-(C6-Pad2)")
+			(net 57 "Net-(C3-Pad2)")
 			(pintype "passive")
 		)
@@
 		(descr "Capacitor SMD 0603 (1608 Metric), square (rectangular) end terminal, IPC_7351 nominal, (Body size source: IPC-SM-782 page 76, https://www.pcb-3d.com/wordpress/wp-content/uploads/ipc-sm-782a_amendment_1_and_2.pdf), generated with kicad-footprint-generator")
 		(tags "capacitor")
-		(property "Reference" "C8"
+		(property "Reference" "C4"
 			(at 0 1.2 90)
 			(unlocked yes)
@@
 			(layers "F.Cu" "F.Paste" "F.Mask")
 			(roundrect_rratio 0.25)
-			(net 57 "Net-(C6-Pad2)")
+			(net 57 "Net-(C3-Pad2)")
 			(pintype "passive")
 		)
@@
 		(descr "FE Package; 16-Lead Plastic TSSOP (4.4mm); Exposed Pad Variation BB; (see Linear Technology 1956f.pdf)")
 		(tags "SSOP 0.65")
-		(property "Reference" "U4"
+		(property "Reference" "U2"
 			(at 4.45 -0.65 0)
 			(unlocked yes)
@@
 		(descr "TSSOP, 14 Pin (JEDEC MO-153 Var AB-1 https://www.jedec.org/document_search?search_api_views_fulltext=MO-153), generated with kicad-footprint-generator ipc_gullwing_generator.py")
 		(tags "TSSOP SO")
-		(property "Reference" "U3"
+		(property "Reference" "U1"
 			(at -4.2 -3.275 0)
 			(unlocked yes)
@@
 			(layers "F.Cu" "F.Paste" "F.Mask")
 			(roundrect_rratio 0.25)
-			(net 95 "Net-(U3-Pad2)")
+			(net 95 "Net-(U1-Pad2)")
 			(pintype "output")
 		)
@@
 			(layers "F.Cu" "F.Paste" "F.Mask")
 			(roundrect_rratio 0.25)
-			(net 95 "Net-(U3-Pad2)")
+			(net 95 "Net-(U1-Pad2)")
 			(pintype "input")
 		)
@@
 			(layers "F.Cu" "F.Paste" "F.Mask")
 			(roundrect_rratio 0.25)
-			(net 95 "Net-(U3-Pad2)")
+			(net 95 "Net-(U1-Pad2)")
 			(pintype "input")
 		)
@@
 			(layers "F.Cu" "F.Paste" "F.Mask")
 			(roundrect_rratio 0.25)
-			(net 98 "unconnected-(U3-Pad8)")
+			(net 98 "unconnected-(U1-Pad8)")
 			(pintype "output+no_connect")
 		)
@@
 			(layers "F.Cu" "F.Paste" "F.Mask")
 			(roundrect_rratio 0.25)
-			(net 96 "unconnected-(U3-Pad10)")
+			(net 96 "unconnected-(U1-Pad10)")
 			(pintype "output+no_connect")
 		)
@@
 			(layers "F.Cu" "F.Paste" "F.Mask")
 			(roundrect_rratio 0.25)
-			(net 97 "unconnected-(U3-Pad12)")
+			(net 97 "unconnected-(U1-Pad12)")
 			(pintype "output+no_connect")
 		)
@@
 		(descr "Capacitor SMD 0603 (1608 Metric), square (rectangular) end terminal, IPC_7351 nominal, (Body size source: IPC-SM-782 page 76, https://www.pcb-3d.com/wordpress/wp-content/uploads/ipc-sm-782a_amendment_1_and_2.pdf), generated with kicad-footprint-generator")
 		(tags "capacitor")
-		(property "Reference" "C5"
-			(at 0 -1.4 90)
+		(property "Reference" "C2"
+			(at 0.625 -1.25 90)
 			(unlocked yes)
 			(layer "B.SilkS")
@@
 		(descr "Capacitor SMD 0603 (1608 Metric), square (rectangular) end terminal, IPC_7351 nominal, (Body size source: IPC-SM-782 page 76, https://www.pcb-3d.com/wordpress/wp-content/uploads/ipc-sm-782a_amendment_1_and_2.pdf), generated with kicad-footprint-generator")
 		(tags "capacitor")
-		(property "Reference" "C4"
+		(property "Reference" "C1"
 			(at 0.05 -1.15 0)
 			(unlocked yes)
@@
 	)
 	(segment
-		(start 136.05 83.2)
-		(end 130.95 78.1)
+		(start 149.35 115.5425)
+		(end 149.35 113.35)
 		(width 0.4)
 		(layer "B.Cu")
@@
 	)
 	(segment
-		(start 151 111.7)
-		(end 151 101.583992)
+		(start 135.95 83.1)
+		(end 130.95 78.1)
 		(width 0.4)
 		(layer "B.Cu")
@@
 	)
 	(segment
-		(start 149.35 115.5425)
-		(end 149.35 113.35)
+		(start 151 101.583992)
+		(end 135.95 86.533992)
 		(width 0.4)
 		(layer "B.Cu")
@@
 	)
 	(segment
-		(start 136.05 86.633992)
-		(end 136.05 83.2)
+		(start 135.95 86.533992)
+		(end 135.95 83.1)
 		(width 0.4)
 		(layer "B.Cu")
@@
 	)
 	(segment
-		(start 149.35 113.35)
-		(end 151 111.7)
+		(start 151 111.7)
+		(end 151 101.583992)
 		(width 0.4)
 		(layer "B.Cu")
@@
 	)
 	(segment
-		(start 151 101.583992)
-		(end 136.05 86.633992)
+		(start 149.35 113.35)
+		(end 151 111.7)
 		(width 0.4)
 		(layer "B.Cu")
@@
 	)
 	(segment
-		(start 156.55 88.5)
+		(start 156.9 88.85)
 		(end 155.2 87.15)
 		(width 0.4)
@@
 	)
 	(via
-		(at 156.55 88.5)
+		(at 156.9 88.85)
 		(size 1)
 		(drill 0.5)
@@
 	)
 	(segment
-		(start 156.55 88.5)
+		(start 156.9 88.85)
 		(end 162.6 94.55)
 		(width 0.4)
@@
 	)
 	(segment
-		(start 157.55 115.9)
-		(end 161.45 112)
+		(start 157 115.85)
+		(end 161.45 111.4)
 		(width 0.4)
 		(layer "F.Cu")
@@
 	)
 	(segment
-		(start 157.55 117)
-		(end 157.55 115.9)
+		(start 157.325 91.175)
+		(end 152.4 86.25)
 		(width 0.4)
 		(layer "F.Cu")
@@
 	)
 	(segment
-		(start 155.3 89.15)
-		(end 152.4 86.25)
+		(start 157 117.55)
+		(end 157 115.85)
 		(width 0.4)
 		(layer "F.Cu")
@@
 	)
 	(segment
-		(start 161.45 112)
-		(end 161.45 100.3)
+		(start 157.375 91.175)
+		(end 157.325 91.175)
 		(width 0.4)
 		(layer "F.Cu")
@@
 	)
 	(segment
-		(start 157 117.55)
-		(end 157.55 117)
+		(start 161.45 111.4)
+		(end 161.45 100.3)
 		(width 0.4)
 		(layer "F.Cu")
@@
 	)
 	(via
-		(at 155.3 89.15)
+		(at 157.375 91.175)
 		(size 1)
 		(drill 0.5)
@@
 	)
 	(segment
-		(start 155.35 89.15)
-		(end 161.45 95.25)
+		(start 156.985 119.2425)
+		(end 156.985 117.565)
 		(width 0.4)
 		(layer "B.Cu")
@@
 	)
 	(segment
-		(start 156.985 119.2425)
-		(end 156.985 117.565)
-		(width 0.4)
-		(layer "B.Cu")
-		(net 46)
-	)
-	(segment
-		(start 155.3 89.15)
-		(end 155.35 89.15)
+		(start 156.985 117.565)
+		(end 157 117.55)
 		(width 0.4)
 		(layer "B.Cu")
@@
 	)
 	(segment
-		(start 156.985 117.565)
-		(end 157 117.55)
+		(start 157.375 91.175)
+		(end 161.45 95.25)
 		(width 0.4)
 		(layer "B.Cu")
