File: kicad/Extension.kicad_sch (KiCad schematic)
At the start: 74 parts, among them J1 FLE-126-01-G-DV, J2 RCJ-044, J3 HDMI A, SW1 PTS645SK43SMTR92 LFS, T1 DA101JC, U3 74HC04, U4 DSLVDS1047

Commit message: Updated PCB
Parts:
- renumbered C4 to C1, C5 to C2, C6 to C3, C8 to C4, U3 to U1, U4 to U2
Changed lines of the file:
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@@
 		(on_board yes)
 		(dnp no)
-		(property "Reference" "#PWR055"
+		(property "Reference" "#PWR047"
 			(at 25.4 252.73 0)
 			(effects
@@
 			(project "ECP5"
 				(path "/968e4a2d-0ddb-4369-8334-6b9cd7c9ac3a/61e66402-2089-43f0-88c3-2a4be23eb1c3"
-					(reference "#PWR055")
+					(reference "#PWR047")
 					(unit 1)
 				)
@@
 		(dnp no)
 		(fields_autoplaced yes)
-		(property "Reference" "C4"
+		(property "Reference" "C1"
 			(at 218.44 194.3162 0)
 			(effects
@@
 			(project "ECP5"
 				(path "/968e4a2d-0ddb-4369-8334-6b9cd7c9ac3a/61e66402-2089-43f0-88c3-2a4be23eb1c3"
-					(reference "C4")
+					(reference "C1")
 					(unit 1)
 				)
@@
 		(on_board yes)
 		(dnp no)
-		(property "Reference" "U3"
+		(property "Reference" "U1"
 			(at 33.02 238.76 0)
 			(effects
@@
 			(project "ECP5"
 				(path "/968e4a2d-0ddb-4369-8334-6b9cd7c9ac3a/61e66402-2089-43f0-88c3-2a4be23eb1c3"
-					(reference "U3")
+					(reference "U1")
 					(unit 4)
 				)
@@
 		(on_board yes)
 		(dnp no)
-		(property "Reference" "U4"
+		(property "Reference" "U2"
 			(at 228.092 199.39 0)
 			(effects
@@
 			(project "ECP5"
 				(path "/968e4a2d-0ddb-4369-8334-6b9cd7c9ac3a/61e66402-2089-43f0-88c3-2a4be23eb1c3"
-					(reference "U4")
+					(reference "U2")
 					(unit 1)
 				)
@@
 		(dnp no)
 		(fields_autoplaced yes)
-		(property "Reference" "U3"
+		(property "Reference" "U1"
 			(at 143.51 234.9499 0)
 			(effects
@@
 			(project "ECP5"
 				(path "/968e4a2d-0ddb-4369-8334-6b9cd7c9ac3a/61e66402-2089-43f0-88c3-2a4be23eb1c3"
-					(reference "U3")
+					(reference "U1")
 					(unit 7)
 				)
@@
 		(on_board yes)
 		(dnp no)
-		(property "Reference" "#PWR051"
+		(property "Reference" "#PWR042"
 			(at 81.28 240.03 0)
 			(effects
@@
 			(project "ECP5"
 				(path "/968e4a2d-0ddb-4369-8334-6b9cd7c9ac3a/61e66402-2089-43f0-88c3-2a4be23eb1c3"
-					(reference "#PWR051")
+					(reference "#PWR042")
 					(unit 1)
 				)
@@
 		(on_board yes)
 		(dnp no)
-		(property "Reference" "#PWR054"
+		(property "Reference" "#PWR041"
 			(at 203.2 232.41 0)
 			(effects
@@
 			(project "ECP5"
 				(path "/968e4a2d-0ddb-4369-8334-6b9cd7c9ac3a/61e66402-2089-43f0-88c3-2a4be23eb1c3"
-					(reference "#PWR054")
+					(reference "#PWR041")
 					(unit 1)
 				)
@@
 		(on_board yes)
 		(dnp no)
-		(property "Reference" "#PWR060"
+		(property "Reference" "#PWR045"
 			(at 227.33 243.84 0)
 			(effects
@@
 			(project "ECP5"
 				(path "/968e4a2d-0ddb-4369-8334-6b9cd7c9ac3a/61e66402-2089-43f0-88c3-2a4be23eb1c3"
-					(reference "#PWR060")
+					(reference "#PWR045")
 					(unit 1)
 				)
@@
 		(on_board yes)
 		(dnp no)
-		(property "Reference" "#PWR039"
+		(property "Reference" "#PWR037"
 			(at 220.98 194.31 0)
 			(effects
@@
 			(project "ECP5"
 				(path "/968e4a2d-0ddb-4369-8334-6b9cd7c9ac3a/61e66402-2089-43f0-88c3-2a4be23eb1c3"
-					(reference "#PWR039")
+					(reference "#PWR037")
 					(unit 1)
 				)
@@
 		(on_board yes)
 		(dnp no)
-		(property "Reference" "#PWR048"
+		(property "Reference" "#PWR040"
 			(at 140.97 229.87 0)
 			(effects
@@
 			(project "ECP5"
 				(path "/968e4a2d-0ddb-4369-8334-6b9cd7c9ac3a/61e66402-2089-43f0-88c3-2a4be23eb1c3"
-					(reference "#PWR048")
+					(reference "#PWR040")
 					(unit 1)
 				)
@@
 		(on_board yes)
 		(dnp no)
-		(property "Reference" "U3"
+		(property "Reference" "U1"
 			(at 52.324 221.488 0)
 			(effects
@@
 			(project "ECP5"
 				(path "/968e4a2d-0ddb-4369-8334-6b9cd7c9ac3a/61e66402-2089-43f0-88c3-2a4be23eb1c3"
-					(reference "U3")
+					(reference "U1")
 					(unit 3)
 				)
@@
 		(on_board yes)
 		(dnp no)
-		(property "Reference" "#PWR047"
+		(property "Reference" "#PWR039"
 			(at 137.16 219.71 0)
 			(effects
@@
 			(project "ECP5"
 				(path "/968e4a2d-0ddb-4369-8334-6b9cd7c9ac3a/61e66402-2089-43f0-88c3-2a4be23eb1c3"
-					(reference "#PWR047")
+					(reference "#PWR039")
 					(unit 1)
 				)
@@
 		(on_board yes)
 		(dnp no)
-		(property "Reference" "#PWR056"
+		(property "Reference" "#PWR048"
 			(at 46.99 252.73 0)
 			(effects
@@
 			(project "ECP5"
 				(path "/968e4a2d-0ddb-4369-8334-6b9cd7c9ac3a/61e66402-2089-43f0-88c3-2a4be23eb1c3"
-					(reference "#PWR056")
+					(reference "#PWR048")
 					(unit 1)
 				)
@@
 		(on_board yes)
 		(dnp no)
-		(property "Reference" "#PWR046"
+		(property "Reference" "#PWR038"
 			(at 220.98 204.47 0)
 			(effects
@@
 			(project "ECP5"
 				(path "/968e4a2d-0ddb-4369-8334-6b9cd7c9ac3a/61e66402-2089-43f0-88c3-2a4be23eb1c3"
-					(reference "#PWR046")
+					(reference "#PWR038")
 					(unit 1)
 				)
@@
 		(on_board yes)
 		(dnp no)
-		(property "Reference" "#PWR053"
+		(property "Reference" "#PWR046"
 			(at 116.84 245.11 0)
 			(effects
@@
 			(project "ECP5"
 				(path "/968e4a2d-0ddb-4369-8334-6b9cd7c9ac3a/61e66402-2089-43f0-88c3-2a4be23eb1c3"
-					(reference "#PWR053")
+					(reference "#PWR046")
 					(unit 1)
 				)
@@
 		(on_board yes)
 		(dnp no)
-		(property "Reference" "#PWR057"
+		(property "Reference" "#PWR049"
 			(at 67.31 252.73 0)
 			(effects
@@
 			(project "ECP5"
 				(path "/968e4a2d-0ddb-4369-8334-6b9cd7c9ac3a/61e66402-2089-43f0-88c3-2a4be23eb1c3"
-					(reference "#PWR057")
+					(reference "#PWR049")
 					(unit 1)
 				)
@@
 		(dnp no)
 		(fields_autoplaced yes)
-		(property "Reference" "C6"
+		(property "Reference" "C3"
 			(at 91.4337 215.9 90)
 			(effects
@@
 			(project "ECP5"
 				(path "/968e4a2d-0ddb-4369-8334-6b9cd7c9ac3a/61e66402-2089-43f0-88c3-2a4be23eb1c3"
-					(reference "C6")
+					(reference "C3")
 					(unit 1)
 				)
@@
 		(on_board yes)
 		(dnp no)
-		(property "Reference" "#PWR059"
+		(property "Reference" "#PWR044"
 			(at 215.9 243.84 0)
 			(effects
@@
 			(project "ECP5"
 				(path "/968e4a2d-0ddb-4369-8334-6b9cd7c9ac3a/61e66402-2089-43f0-88c3-2a4be23eb1c3"
-					(reference "#PWR059")
+					(reference "#PWR044")
 					(unit 1)
 				)
@@
 		(on_board yes)
 		(dnp no)
-		(property "Reference" "#PWR052"
+		(property "Reference" "#PWR043"
 			(at 97.79 240.03 0)
 			(effects
@@
 			(project "ECP5"
 				(path "/968e4a2d-0ddb-4369-8334-6b9cd7c9ac3a/61e66402-2089-43f0-88c3-2a4be23eb1c3"
-					(reference "#PWR052")
+					(reference "#PWR043")
 					(unit 1)
 				)
@@
 		(on_board yes)
 		(dnp no)
-		(property "Reference" "U3"
+		(property "Reference" "U1"
 			(at 52.07 208.534 0)
 			(effects
@@
 			(project "ECP5"
 				(path "/968e4a2d-0ddb-4369-8334-6b9cd7c9ac3a/61e66402-2089-43f0-88c3-2a4be23eb1c3"
-					(reference "U3")
+					(reference "U1")
 					(unit 2)
 				)
@@
 		(on_board yes)
 		(dnp no)
-		(property "Reference" "U3"
+		(property "Reference" "U1"
 			(at 54.61 239.014 0)
 			(effects
@@
 			(project "ECP5"
 				(path "/968e4a2d-0ddb-4369-8334-6b9cd7c9ac3a/61e66402-2089-43f0-88c3-2a4be23eb1c3"
-					(reference "U3")
+					(reference "U1")
 					(unit 5)
 				)
@@
 		(on_board yes)
 		(dnp no)
-		(property "Reference" "#PWR058"
+		(property "Reference" "#PWR050"
 			(at 137.16 255.27 0)
 			(effects
@@
 			(project "ECP5"
 				(path "/968e4a2d-0ddb-4369-8334-6b9cd7c9ac3a/61e66402-2089-43f0-88c3-2a4be23eb1c3"
-					(reference "#PWR058")
+					(reference "#PWR050")
 					(unit 1)
 				)
@@
 		(on_board yes)
 		(dnp no)
-		(property "Reference" "#PWR061"
+		(property "Reference" "#PWR051"
 			(at 287.02 266.7 0)
 			(effects
@@
 			(project "ECP5"
 				(path "/968e4a2d-0ddb-4369-8334-6b9cd7c9ac3a/61e66402-2089-43f0-88c3-2a4be23eb1c3"
-					(reference "#PWR061")
+					(reference "#PWR051")
 					(unit 1)
 				)
@@
 		(on_board yes)
 		(dnp no)
-		(property "Reference" "U3"
+		(property "Reference" "U1"
 			(at 74.93 238.506 0)
 			(effects
@@
 			(project "ECP5"
 				(path "/968e4a2d-0ddb-4369-8334-6b9cd7c9ac3a/61e66402-2089-43f0-88c3-2a4be23eb1c3"
-					(reference "U3")
+					(reference "U1")
 					(unit 6)
 				)
@@
 		(dnp no)
 		(fields_autoplaced yes)
-		(property "Reference" "C5"
+		(property "Reference" "C2"
 			(at 143.51 219.7162 0)
 			(effects
@@
 			(project "ECP5"
 				(path "/968e4a2d-0ddb-4369-8334-6b9cd7c9ac3a/61e66402-2089-43f0-88c3-2a4be23eb1c3"
-					(reference "C5")
+					(reference "C2")
 					(unit 1)
 				)
@@
 		(on_board yes)
 		(dnp no)
-		(property "Reference" "C8"
+		(property "Reference" "C4"
 			(at 118.11 234.442 0)
 			(effects
@@
 			(project "ECP5"
 				(path "/968e4a2d-0ddb-4369-8334-6b9cd7c9ac3a/61e66402-2089-43f0-88c3-2a4be23eb1c3"
-					(reference "C8")
+					(reference "C4")
 					(unit 1)
 				)
@@
 		(on_board yes)
 		(dnp no)
-		(property "Reference" "U3"
+		(property "Reference" "U1"
 			(at 33.02 214.884 0)
 			(effects
@@
 			(project "ECP5"
 				(path "/968e4a2d-0ddb-4369-8334-6b9cd7c9ac3a/61e66402-2089-43f0-88c3-2a4be23eb1c3"
-					(reference "U3")
+					(reference "U1")
 					(unit 1)
 				)

Commit message: Added measurements
Other:
- note added: "COAX"
- note added: "Measured: 1Vpp"
- note added: "Measured: W/ no load 1Vpp"
- note removed: "RCA"
Changed lines of the file:
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@@
 		)
 	)
-	(text "RCA"
+	(text "COAX"
 		(exclude_from_sim no)
 		(at 19.05 188.468 0)
@@
 		)
 	)
+	(text "Measured: W/ no load 1Vpp"
+		(exclude_from_sim no)
+		(at 114.3 206.756 0)
+		(effects
+			(font
+				(size 1.27 1.27)
+			)
+		)
+	)
 	(text "96KHZ"
 		(exclude_from_sim no)
@@
 		(effects
 			(font
+				(size 1.27 1.27)
+			)
+		)
+	)
+	(text "Measured: 1Vpp"
+		(exclude_from_sim no)
+		(at 81.788 206.756 0)
+		(effects
+			(font
